File: Hardware/Controller/Controller.kicad_pcb (KiCad board)
At the start: 2 copper layers, 28 x 38 mm, 17 parts, among them J1 Conn_02x06_Odd_Even, J2 Conn_01x05_Female, J3 Conn_01x02_Male, J4 Conn_01x02_Male, J5 Conn_01x02_Male, J6 Conn_01x02_Male, SW1 SW_SPST, SW3 SW_SPST, SW4 SW_SPST, SW5 SW_SPST

Commit message: rev 2 Hw
Parts:
- turned D1 to 90 degrees
- turned D2 to 90 degrees
- turned D3 to 90 degrees
- turned D4 to 90 degrees
- turned D5 to 90 degrees
- turned D6 to 90 degrees
Connections:
- D1 pad 1: /CON_BM1 -> Net-(D1-Pad1)
- D1 pad 2: Net-(D1-Pad2) -> /CON_BM1
- D2 pad 1: /CON_BM1 -> Net-(D2-Pad1)
- D2 pad 2: Net-(D2-Pad2) -> /CON_BM1
- D3 pad 1: /CON_BM1 -> Net-(D3-Pad1)
- D3 pad 2: Net-(D3-Pad2) -> /CON_BM1
- D4 pad 1: /CON_BM2 -> Net-(D4-Pad1)
- D4 pad 2: Net-(D4-Pad2) -> /CON_BM2
- D5 pad 1: /CON_BM2 -> Net-(D5-Pad1)
- D5 pad 2: Net-(D5-Pad2) -> /CON_BM2
- D6 pad 1: /CON_BM2 -> Net-(D6-Pad1)
- D6 pad 2: Net-(D6-Pad2) -> /CON_BM2
- J1 pad 4: (no net) -> /CON_SPEZ
- J5 pad 1: Net-(D3-Pad2) -> Net-(D3-Pad1)
- J6 pad 2: Net-(D6-Pad2) -> Net-(D6-Pad1)
- SW1 pad 1: Net-(D2-Pad2) -> Net-(D2-Pad1)
- SW3 pad 2: Net-(D4-Pad2) -> Net-(D4-Pad1)
- SW4 pad 1: Net-(D1-Pad2) -> Net-(D1-Pad1)
- SW5 pad 2: Net-(D5-Pad2) -> Net-(D5-Pad1)
Routing:
- net Net-(D2-Pad2): track 16.5 -> 0.00 mm
- net Net-(D2-Pad1): track 0.00 -> 16.5 mm
- net Net-(D5-Pad2): track 14.0 -> 0.00 mm
- net Net-(D5-Pad1): track 0.00 -> 14.0 mm
- net Net-(D4-Pad2): track 12.4 -> 0.00 mm
- net Net-(D4-Pad1): track 0.00 -> 12.4 mm
- net Net-(D1-Pad2): track 11.3 -> 0.00 mm
- net Net-(D1-Pad1): track 0.00 -> 11.3 mm
- net Net-(D6-Pad2): track 4.77 -> 0.00 mm
- net Net-(D6-Pad1): track 0.00 -> 4.77 mm
- net Net-(D3-Pad2): track 3.56 -> 0.00 mm
- net Net-(D3-Pad1): track 0.00 -> 3.56 mm
Other:
- net class Default removed
- board text added: "Controller Rev B"
- board text added: "Pixeldeck"
- board text removed: "Controller Rev A"
- board text removed: "H-HTV-Matrix"
