File: Hardware/Mainboard/Mainboard.kicad_pcb (KiCad board)
At the start: 2 copper layers, 70 x 45.1 mm, 46 parts, among them J1 Conn_01x05, J2 Conn_02x08_Odd_Even, J3 Conn_02x06_Odd_Even, J4 Conn_02x06_Odd_Even, J5 Conn_02x02_Odd_Even, J6 Conn_01x04, J7 Conn_01x02, J8 Conn_01x02, J9 Conn_01x04, Q1 BSS123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

Commit message: rev 2 Hw
Parts:
- added R12: 10k, Resistor_SMD:R_0402_1005Metric, F.Cu at (151.1, 64.9)
- added R13: 33k, Resistor_SMD:R_0402_1005Metric, F.Cu at (140.3, 76.8)
- added R14: 10k, Resistor_SMD:R_0402_1005Metric, F.Cu at (146.8, 42.2)
- added R15: 10k, Resistor_SMD:R_0402_1005Metric, F.Cu at (148.5, 42.2)
- C17: footprint Capacitor_SMD:C_0402_1005Metric -> Capacitor_SMD:C_1210_3225Metric
- Q1: value BSS123 -> HD2302
- moved C17 1.78 mm to (120.1, 47.5)
- moved J1 0.56 mm to (145.3, 49.1)
Connections:
- U1 pad 17: (no net) -> unconnected-(U1-Pad17)
- U1 pad 18: (no net) -> unconnected-(U1-Pad18)
- U1 pad 19: (no net) -> unconnected-(U1-Pad19)
- U1 pad 20: (no net) -> unconnected-(U1-Pad20)
- U1 pad 21: (no net) -> unconnected-(U1-Pad21)
- U1 pad 22: (no net) -> unconnected-(U1-Pad22)
- U1 pad 32: (no net) -> unconnected-(U1-Pad32)
- U1 pad 36: (no net) -> Net-(U1-Pad36)
- U1 pad 37: (no net) -> Net-(U1-Pad37)
- U1 pad 4: (no net) -> unconnected-(U1-Pad4)
- U1 pad 5: (no net) -> unconnected-(U1-Pad5)
- U1 pad 6: (no net) -> unconnected-(U1-Pad6)
- U1 pad 7: (no net) -> unconnected-(U1-Pad7)
- U2 pad 12: (no net) -> unconnected-(U2-Pad12)
- U2 pad 13: (no net) -> /RCON_JB
- U2 pad 2: (no net) -> unconnected-(U2-Pad2)
- U2 pad 3: (no net) -> unconnected-(U2-Pad3)
- U2 pad 36: (no net) -> unconnected-(U2-Pad36)
- U2 pad 37: (no net) -> unconnected-(U2-Pad37)
- U2 pad 44: (no net) -> unconnected-(U2-Pad44)
- U3 pad 3: /KEEPALIVE -> Net-(U3-Pad3)
Routing:
- net /PDI_DATA: track 5.87 -> 52.3 mm, vias 0 -> 2
- net /PDI_CLK: track 7.49 -> 52.3 mm, vias 0 -> 2
- net /RCON_JB: track 25.5 -> 39.0 mm
- net Net-(U1-Pad37): track 0.00 -> 8.45 mm
- net -BATT: track 47.3 -> 39.6 mm, vias 84 -> 80
- net Net-(U1-Pad36): track 0.00 -> 7.07 mm
- net /KEEPALIVE: track 32.7 -> 29.8 mm, vias 3 -> 2
- net +VSW: track 19.5 -> 22.1 mm
- net Net-(U3-Pad3): track 0.00 -> 1.84 mm
Other:
- net class Default removed
- net class Power removed
- board text added: "Pixeldeck"
- board text added: "Rev B"
- board text added: "by Lars and Finn 19.02.23"
- board text added: "htv"
- board text removed: "H-HTV-Matrix"
- board text removed: "Rev A"
- board text removed: "by Lars"
